File: PCB/tamagotchi.kicad_pcb (KiCad board)
At the start: 2 copper layers, 56.8 x 66.2 mm, 14 parts, among them SW1 SW_Push, SW2 SW_Push, SW3 SW_Push, U1 XIAO-ESP32-C6, U2 HS96L03W2C03

Commit message: Refactor code structure for improved readability and maintainability
Parts:
- renumbered VBAT to TP1, GND to TP2
Routing:
- net Net-(U1-GPIO2/A2/D2): track 11.2 -> 13.0 mm
- net GND: vias 274 -> 271
